Commit message: 更新训练： 1.初步使用s54跑起来训练 2.跑起来训练暂时去掉了一些惩罚奖励、提高了kp值，使用的是Tienkung转换过去的数据，后续这些项需要排查去除

File: legged_lab/assets/biped_s54/urdf/biped_s54.urdf (robot description, URDF)
Before this commit: robot biped_s54, 33 links, 32 joints
Links:
- removed link waist_yaw
- added link dummy_link
- added link head_rader, mass 0.26500; visual mesh filename=../meshes/head_rader.STL
- added link l_foot_heel; collision sphere radius=0.005
- added link l_foot_toe; collision sphere radius=0.005
- added link ll_foot_heel; collision sphere radius=0.005
- added link ll_foot_toe; collision sphere radius=0.005
- added link lr_foot_heel; collision sphere radius=0.005
- added link lr_foot_toe; collision sphere radius=0.005
- added link r_foot_heel; collision sphere radius=0.005
- added link r_foot_toe; collision sphere radius=0.005
- added link rl_foot_heel; collision sphere radius=0.005
- added link rl_foot_toe; collision sphere radius=0.005
- added link rr_foot_heel; collision sphere radius=0.005
- added link rr_foot_toe; collision sphere radius=0.005
- added link waist_camera, mass 0.13300; visual mesh filename=../meshes/waist_camera.STL
- added link waist_yaw_link, mass 20.23838; visual mesh filename=../meshes/waist_yaw.STL
- link base_link: mass 7.06405 -> 7.54373; geometry collision box size=0.25 0.32 0.37; visual mesh filename=../meshes/torso.STL
- link camera_base: mass 0.0482361371130408 -> 0.00000000
- link leg_l1_link: mass 1.55641 -> 1.56067
- link leg_l2_link: mass 0.75873 -> 0.77767
- link leg_l3_link: mass 6.68074 -> 6.52432; geometry collision box size=0.12 0.1 0.2; visual mesh filename=../meshes/l_leg_pitch.STL
- link leg_l4_link: mass 3.64666 -> 3.55159; geometry collision box size=0.08 0.08 0.1; visual mesh filename=../meshes/l_knee.STL
- link leg_l5_link: mass 0.07848 -> 0.07554
- link leg_l6_link: mass 0.69242 -> 0.60538; geometry visual mesh filename=../meshes/l_foot_roll.STL
- link leg_r1_link: mass 1.55641 -> 1.56067
- link leg_r2_link: mass 0.75873 -> 0.77767
- link leg_r3_link: mass 6.68074 -> 6.52432; geometry collision box size=0.12 0.1 0.2; visual mesh filename=../meshes/r_leg_pitch.STL
- link leg_r4_link: mass 3.64666 -> 3.55159; geometry collision box size=0.08 0.08 0.1; visual mesh filename=../meshes/r_knee.STL
- link leg_r5_link: mass 0.07848 -> 0.07554
- link leg_r6_link: mass 0.69242 -> 0.60538; geometry visual mesh filename=../meshes/r_foot_roll.STL
- link zarm_l1_link: mass 0.94521 -> 0.96332
- link zarm_l2_link: mass 0.41921 -> 0.44946
- link zarm_l3_link: mass 1.78857 -> 1.83951; geometry collision cylinder length=0.15 radius=0.06; visual mesh filename=../meshes/l_arm_yaw.STL
- link zarm_l4_link: mass 0.63149 -> 0.66448; geometry collision cylinder length=0.15 radius=0.058; visual mesh filename=../meshes/l_forearm.STL
- link zarm_l5_link: mass 0.60828 -> 0.67508
- link zarm_l6_link: mass 0.50616 -> 0.51484
- link zarm_l7_end_effector: geometry collision box size=0.12 0.10 0.235
- link zarm_l7_link: mass 0.18940 -> 0.7374; geometry visual mesh filename=../meshes/l_hand_pitch_nohand.STL
- link zarm_r1_link: mass 0.92947 -> 0.96332
- link zarm_r2_link: mass 0.41523 -> 0.44946
- link zarm_r3_link: mass 1.78473 -> 1.83951; geometry collision cylinder length=0.15 radius=0.06; visual mesh filename=../meshes/r_arm_yaw.STL
- link zarm_r4_link: mass 0.63548 -> 0.66448; geometry collision cylinder length=0.15 radius=0.058; visual mesh filename=../meshes/r_forearm.STL
- link zarm_r5_link: mass 0.61021 -> 0.67508
- link zarm_r6_link: mass 0.53821 -> 0.51484
- link zarm_r7_end_effector: geometry collision box size=0.12 0.10 0.235
- link zarm_r7_link: mass 0.19960 -> 0.7374; geometry visual mesh filename=../meshes/r_hand_pitch_nohand.STL
- link zhead_1_link: mass 0.57250 -> 0.55195
- link zhead_2_link: mass 0.73448 -> 0.82380
Joints:
- added joint dummy_to_base_link: type fixed, parent dummy_link, child base_link, origin xyz=0 0 0 rpy=0 0 0
- added joint head_rader_joint: type fixed, parent zhead_1_link, child head_rader, origin xyz=0 0 -0.078253 rpy=0 0 0, axis 0 0 0
- added joint l_foot_heel_joint: type fixed, parent leg_l6_link, child l_foot_heel, origin xyz=-0.073164 0.0 -0.0595 rpy=0 0 0
- added joint l_foot_toe_joint: type fixed, parent leg_l6_link, child l_foot_toe, origin xyz=0.17084 0.0 -0.0595 rpy=0 0 0
- added joint ll_foot_heel_joint: type fixed, parent leg_l6_link, child ll_foot_heel, origin xyz=-0.073164 0.05 -0.0595 rpy=0 0 0
- added joint ll_foot_toe_joint: type fixed, parent leg_l6_link, child ll_foot_toe, origin xyz=0.17084 0.05 -0.0595 rpy=0 0 0
- added joint lr_foot_heel_joint: type fixed, parent leg_l6_link, child lr_foot_heel, origin xyz=-0.073164 -0.05 -0.0595 rpy=0 0 0
- added joint lr_foot_toe_joint: type fixed, parent leg_l6_link, child lr_foot_toe, origin xyz=0.17084 -0.05 -0.0595 rpy=0 0 0
- added joint r_foot_heel_joint: type fixed, parent leg_r6_link, child r_foot_heel, origin xyz=-0.073164 0.0 -0.0595 rpy=0 0 0
- added joint r_foot_toe_joint: type fixed, parent leg_r6_link, child r_foot_toe, origin xyz=0.17084 0.0 -0.0595 rpy=0 0 0
- added joint rl_foot_heel_joint: type fixed, parent leg_r6_link, child rl_foot_heel, origin xyz=-0.073164 0.05 -0.0595 rpy=0 0 0
- added joint rl_foot_toe_joint: type fixed, parent leg_r6_link, child rl_foot_toe, origin xyz=0.17084 0.05 -0.0595 rpy=0 0 0
- added joint rr_foot_heel_joint: type fixed, parent leg_r6_link, child rr_foot_heel, origin xyz=-0.073164 -0.05 -0.0595 rpy=0 0 0
- added joint rr_foot_toe_joint: type fixed, parent leg_r6_link, child rr_foot_toe, origin xyz=0.17084 -0.05 -0.0595 rpy=0 0 0
- added joint waist_camera: type fixed, parent waist_yaw_link, child waist_camera, origin xyz=0.0787 0 -0.028449 rpy=0 0.59341 0, axis 0 0 0
- joint camera_base: origin xyz=0.119717018973535 0.0237514612535074 0.0262044145991832 rpy=0 0.480224871300295 0 -> xyz=0.093839 0.0475 0.050077 rpy=0 0.3406 0
- joint leg_l1_joint: limit lower=-0.314159265358979 upper=0.663225115757845 effort=180.0 velocity=23.55 -> lower=-0.314159265358979 upper=0.663225115757845 effort=127.0 velocity=10.4
- joint leg_l2_joint: limit lower=-0.872664625997165 upper=0.785398163397448 effort=100.0 velocity=41.3433333333333 -> lower=-0.785398163397448 upper=1.91986217719376 effort=71.0 velocity=8.7
- joint leg_l3_joint: limit lower=-2.00712863979348 upper=1.5707963267949 effort=100.0 velocity=41.3433333333333 -> lower=-1.91986217719376 upper=1.5707963267949 effort=132 velocity=12.7
- joint leg_l4_joint: limit lower=0.0 upper=2.53072741539178 effort=180.0 velocity=23.55 -> lower=0.0 upper=2.53072741539178 effort=280.0 velocity=10.4
- joint leg_l5_joint: limit lower=-0.872664625997165 upper=0.349065850398866 effort=102.6 velocity=17.8 -> lower=-0.872664625997165 upper=0.349065850398866 effort=91.6 velocity=17.8
- joint leg_l6_joint: limit lower=-0.261799387799149 upper=0.261799387799149 effort=102.6 velocity=17.8 -> lower=-0.261799387799149 upper=0.261799387799149 effort=30.0 velocity=17.8
- joint leg_r2_joint: limit lower=-0.785398163397448 upper=0.872664625997165 effort=100.0 velocity=41.3433333333333 -> lower=-1.91986217719376 upper=0.785398163397448 effort=71.0 velocity=8.7
- joint leg_r3_joint: limit lower=-2.00712863979348 upper=1.5707963267949 effort=100.0 velocity=41.3433333333333 -> lower=-1.91986217719376 upper=1.5707963267949 effort=132.0 velocity=12.7
- joint leg_r4_joint: limit lower=0.0 upper=2.53072741539178 effort=180.0 velocity=23.55 -> lower=0.0 upper=2.53072741539178 effort=280.0 velocity=10.4; origin xyz=0 0 -0.284 rpy=0 0 0 -> xyz=-0.0011639 0 -0.284 rpy=0 0 0
- joint leg_r5_joint: limit lower=-0.872664625997165 upper=0.349065850398866 effort=102.6 velocity=17.8 -> lower=-0.872664625997165 upper=0.349065850398866 effort=91.6 velocity=17.8; origin xyz=0.00199999999983541 -0.000300000028212572 -0.415999999987417 rpy=0 0 0 -> xyz=0.002 0 -0.416 rpy=0 0 0
- joint leg_r6_joint: limit lower=-0.261799387799149 upper=0.261799387799149 effort=102.6 velocity=17.8 -> lower=-0.261799387799149 upper=0.261799387799149 effort=30.0 velocity=17.8
- joint waist_yaw_joint: child waist_yaw -> waist_yaw_link
- joint zarm_l1_joint: parent waist_yaw -> waist_yaw_link
- joint zarm_l7_end_effector_joint: origin xyz=0 -0.03 -0.17 rpy=0 0 0 -> xyz=0 0.0 -0.17 rpy=0 0 0
- joint zarm_r1_joint: parent waist_yaw -> waist_yaw_link
- joint zarm_r7_end_effector_joint: origin xyz=0 0.03 -0.17 rpy=0 0 0 -> xyz=0 0.0 -0.17 rpy=0 0 0
- joint zhead_1_joint: parent waist_yaw -> waist_yaw_link

File: legged_lab/assets/biped_s54/urdf/drake/biped_v3.urdf (robot description, URDF)
Before this commit: robot biped_v3, 14 links, 13 joints
Links:
- removed link waist_yaw
- added link waist_yaw_link, mass 33.70028; visual mesh filename=../../meshes/waist_yaw.STL
- link leg_l1_link: mass 1.63858534 -> 1.56067
- link leg_l2_link: mass 0.70575545 -> 0.77767
- link leg_l3_link: mass 5.93791258 -> 6.52432
- link leg_l4_link: mass 4.02498548 -> 3.55159
- link leg_l5_link: mass 0.07848005 -> 0.07554
- link leg_l6_link: mass 0.58491513 -> 0.60538
- link leg_r1_link: mass 1.63861324 -> 1.56067
- link leg_r2_link: mass 0.70575545 -> 0.77767
- link leg_r3_link: mass 5.93791831 -> 6.52432
- link leg_r4_link: mass 4.02498548 -> 3.55159
- link leg_r5_link: mass 0.07848005 -> 0.07554
- link leg_r6_link: mass 0.58491513 -> 0.60538
- link torso: mass 18.99013928 -> 7.54373; geometry visual mesh filename=../../meshes/torso.STL
Joints:
- removed joint waist_yaw
- added joint waist_yaw_joint: type fixed, parent torso, child waist_yaw_link, origin xyz=0 0 0.1114 rpy=0 0 0, axis 0 0 1, limit lower=-3.14159 upper=3.14159 effort=102.0 velocity=8.7
- joint leg_l1_joint: limit lower=-0.314159265358979 upper=0.663225115757845 effort=180.0 velocity=23.55 -> lower=-0.314159265358979 upper=0.663225115757845 effort=127.0 velocity=10.4
- joint leg_l2_joint: limit lower=-1.91986217719376 upper=0.785398163397448 effort=100.0 velocity=41.3433333333333 -> lower=-0.785398163397448 upper=1.91986217719376 effort=71.0 velocity=8.7
- joint leg_l3_joint: limit lower=-1.91986217719376 upper=1.5707963267949 effort=100.0 velocity=41.3433333333333 -> lower=-1.91986217719376 upper=1.5707963267949 effort=132 velocity=12.7
- joint leg_l4_joint: limit lower=0.0 upper=2.53072741539178 effort=180.0 velocity=23.55 -> lower=0.0 upper=2.53072741539178 effort=280.0 velocity=10.4; origin xyz=0 0 -0.284 rpy=0 0 0 -> xyz=-0.0011639 0 -0.284 rpy=0 0 0
- joint leg_l5_joint: limit lower=-0.872664625997165 upper=0.349065850398866 effort=36.0 velocity=23.0266666666667 -> lower=-0.872664625997165 upper=0.349065850398866 effort=91.6 velocity=17.8; origin xyz=0.002 0.0003 -0.416 rpy=0 0 0 -> xyz=0.002 0 -0.416 rpy=0 0 0
- joint leg_l6_joint: limit lower=-0.261799387799149 upper=0.261799387799149 effort=36.0 velocity=23.0266666666667 -> lower=-0.261799387799149 upper=0.261799387799149 effort=30.0 velocity=17.8
- joint leg_r1_joint: limit lower=-0.663225115757845 upper=0.314159265358979 effort=180.0 velocity=23.55 -> lower=-0.663225115757845 upper=0.314159265358979 effort=127.0 velocity=10.4
- joint leg_r2_joint: limit lower=-0.785398163397448 upper=1.91986217719376 effort=100.0 velocity=41.3433333333333 -> lower=-1.91986217719376 upper=0.785398163397448 effort=71.0 velocity=8.7
- joint leg_r3_joint: limit lower=-1.91986217719376 upper=1.5707963267949 effort=100.0 velocity=41.3433333333333 -> lower=-1.91986217719376 upper=1.5707963267949 effort=132.0 velocity=12.7
- joint leg_r4_joint: limit lower=0.0 upper=2.53072741539178 effort=180.0 velocity=23.55 -> lower=0.0 upper=2.53072741539178 effort=280.0 velocity=10.4; origin xyz=0 0 -0.284 rpy=0 0 0 -> xyz=-0.0011639 0 -0.284 rpy=0 0 0
- joint leg_r5_joint: limit lower=-0.872664625997165 upper=0.349065850398866 effort=36.0 velocity=23.0266666666667 -> lower=-0.872664625997165 upper=0.349065850398866 effort=91.6 velocity=17.8; origin xyz=0.00199999999983541 -0.000300000028212572 -0.415999999987417 rpy=0 0 0 -> xyz=0.002 0 -0.416 rpy=0 0 0
- joint leg_r6_joint: limit lower=-0.261799387799149 upper=0.261799387799149 effort=36.0 velocity=23.0266666666667 -> lower=-0.261799387799149 upper=0.261799387799149 effort=30.0 velocity=17.8

File: legged_lab/assets/biped_s54/urdf/drake/biped_v3_all_joint.urdf (robot description, URDF)
Before this commit: robot biped_v3_all_joint, 35 links, 30 joints
Links:
- link torso: mass 33.93314316 -> 38.42194316

File: legged_lab/assets/biped_s54/urdf/drake/biped_v3_arm.urdf (robot description, URDF)
Before this commit: robot biped_s45, 17 links, 16 joints
Links:
- added link waist_yaw_link, mass 17.39118; visual mesh filename=../../meshes/waist_yaw.STL
- link base_link: mass 22.11293803 -> 7.54373; geometry visual mesh filename=../../meshes/torso.STL
- link zarm_l1_link: mass 0.962 -> 0.96332
- link zarm_l2_link: mass 0.57 -> 0.44946
- link zarm_l3_link: mass 1.65 -> 1.83951
- link zarm_l4_link: mass 0.429 -> 0.66448
- link zarm_l5_link: mass 0.61 -> 0.67508
- link zarm_l6_link: mass 0.331 -> 0.51484
- link zarm_l7_end_effector: geometry 
- link zarm_l7_link: mass 0.64 -> 0.7374; geometry visual mesh filename=../../meshes/l_hand_pitch_nohand.STL
- link zarm_r1_link: mass 0.962 -> 0.96332
- link zarm_r2_link: mass 0.57 -> 0.44946
- link zarm_r3_link: mass 1.65 -> 1.83951
- link zarm_r4_link: mass 0.429 -> 0.66448
- link zarm_r5_link: mass 0.61 -> 0.67508
- link zarm_r6_link: mass 0.331 -> 0.51484
- link zarm_r7_end_effector: geometry 
- link zarm_r7_link: mass 0.64 -> 0.7374; geometry visual mesh filename=../../meshes/r_hand_pitch_nohand.STL
Joints:
- added joint waist_yaw_joint: type fixed, parent base_link, child waist_yaw_link, origin xyz=0 0 0.1114 rpy=0 0 0, axis 0 0 1, limit lower=-3.14159 upper=3.14159 effort=102.0 velocity=8.7
- joint zarm_l1_joint: limit lower=-3.14159265358979 upper=1.5707963267949 effort=100.0 velocity=41.3433333333333 -> lower=-3.14159265358979 upper=1.5707963267949 effort=66.0 velocity=18.8; origin xyz=-0.017499853 0.29269999999999996 0.4245 rpy=0 0 0 -> xyz=-0.003 0.2527 0.283 rpy=0 0 0; parent base_link -> waist_yaw_link
- joint zarm_l2_joint: limit lower=-0.349065850398866 upper=2.0943951023932 effort=50.0 velocity=19.154 -> lower=-0.349065850398866 upper=3.49065850398866 effort=75.0 velocity=8.0
- joint zarm_l3_joint: limit lower=-1.5707963267949 upper=1.5707963267949 effort=39.0 velocity=18.84 -> lower=-1.48352986419518 upper=1.48352986419518 effort=57.0 velocity=7.5
- joint zarm_l4_joint: limit lower=-2.61799387799149 upper=0.0 effort=50.0 velocity=18.84 -> lower=-2.61799387799149 upper=0.0 effort=75.0 velocity=8.0; origin xyz=0.0200000000000006 0 -0.283699999999996 rpy=0 0 0 -> xyz=0.02 0 -0.2837 rpy=0 0 0
- joint zarm_l5_joint: limit lower=-1.5707963267949 upper=1.5707963267949 effort=12.0 velocity=21.666 -> lower=-1.5707963267949 upper=1.5707963267949 effort=14.1 velocity=17.5; origin xyz=-0.0200000000000025 0 -0.127037274261591 rpy=0 0 0 -> xyz=-0.02 0 -0.1201 rpy=0 0 0
- joint zarm_l6_joint: limit lower=-1.30899693899575 upper=0.698131700797732 effort=12.0 velocity=21.666 -> lower=-1.30899693899575 upper=0.698131700797732 effort=14.1 velocity=17.5; origin xyz=0.000199999999999079 0 -0.106462725738415 rpy=0 0 0 -> xyz=0.0 0 -0.114 rpy=0 0 0
- joint zarm_l7_end_effector_joint: origin xyz=0 -0.03 -0.17 rpy=0 0 0 -> xyz=0 0.0 -0.17 rpy=0 0 0
- joint zarm_l7_joint: limit lower=-0.698131700797732 upper=0.698131700797732 effort=12.0 velocity=21.666 -> lower=-0.698131700797732 upper=0.698131700797732 effort=14.1 velocity=17.5; origin xyz=0 0 -0.0210004653879916 rpy=0 0 0 -> xyz=0 0 -0.021 rpy=0 0 0
- joint zarm_r1_joint: limit lower=-3.14159265358979 upper=1.5707963267949 effort=100.0 velocity=41.3433333333333 -> lower=-3.14159265358979 upper=1.5707963267949 effort=66.0 velocity=18.8; origin xyz=-0.017499853 -0.29269999999999996 0.4245 rpy=0 0 0 -> xyz=-0.003 -0.2527 0.283 rpy=0 0 0; parent base_link -> waist_yaw_link
- joint zarm_r2_joint: limit lower=-2.0943951023932 upper=0.349065850398866 effort=50.0 velocity=19.154 -> lower=-3.49065850398866 upper=0.349065850398866 effort=75.0 velocity=8.0
- joint zarm_r3_joint: limit lower=-1.5707963267949 upper=1.5707963267949 effort=39.0 velocity=18.84 -> lower=-1.48352986419518 upper=1.48352986419518 effort=57.0 velocity=7.5
- joint zarm_r4_joint: limit lower=-2.61799387799149 upper=0.0 effort=50.0 velocity=18.84 -> lower=-2.61799387799149 upper=0.0 effort=75.0 velocity=8.0; origin xyz=0.0200000000000024 0 -0.2837 rpy=0 0 0 -> xyz=0.02 0 -0.2837 rpy=0 0 0
- joint zarm_r5_joint: limit lower=-1.5707963267949 upper=1.5707963267949 effort=12.0 velocity=21.666 -> lower=-1.5707963267949 upper=1.5707963267949 effort=14.1 velocity=17.5; origin xyz=-0.0200000000000001 0 -0.127037274261587 rpy=0 0 0 -> xyz=-0.02 0 -0.1201 rpy=0 0 0
- joint zarm_r6_joint: limit lower=-0.698131700797732 upper=1.30899693899575 effort=12.0 velocity=21.666 -> lower=-0.698131700797732 upper=1.30899693899575 effort=14.1 velocity=17.5; origin xyz=0 0 -0.106462725738415 rpy=0 0 0 -> xyz=0.0 0 -0.114 rpy=0 0 0
- joint zarm_r7_end_effector_joint: origin xyz=0 0.03 -0.17 rpy=0 0 0 -> xyz=0 0.0 -0.17 rpy=0 0 0
- joint zarm_r7_joint: limit lower=-0.698131700797732 upper=0.698131700797732 effort=12.0 velocity=21.666 -> lower=-0.698131700797732 upper=0.698131700797732 effort=14.1 velocity=17.5; origin xyz=0 0 -0.0209999999999999 rpy=0 0 0 -> xyz=0.0 0 -0.021 rpy=0 0 0
