Commit message: 更新训练： 1.初步使用s54跑起来训练 2.跑起来训练暂时去掉了一些惩罚奖励、提高了kp值，使用的是Tienkung转换过去的数据，后续这些项需要排查去除

File: legged_lab/assets/biped_s54/urdf/drake/biped_v3_full.urdf (robot description, URDF)
Before this commit: robot biped_v3_full, 28 links, 27 joints
Links:
- removed link torso
- removed link waist_yaw
- added link base_link, mass 6.48663928; visual mesh filename=../../meshes/base_link.STL
- added link dummy_link
- added link head_camera, mass 0.0400617267216207; visual mesh filename=../../meshes/head_camera.STL
- added link waist_yaw_link, mass 22.55935568; visual mesh filename=../../meshes/waist_yaw.STL
- added link zhead_1_link, mass 0.87117795; visual mesh filename=../../meshes/head_yaw.STL
- added link zhead_2_link, mass 0.80529305; visual mesh filename=../../meshes/head_pitch.STL
- link leg_l1_link: mass 1.71093115 -> 1.63858534
- link leg_l2_link: mass 0.58029165 -> 0.70575545
- link leg_l3_link: mass 4.50393141 -> 5.93791258
- link leg_l4_link: mass 1.62776815 -> 4.02498548
- link leg_l5_link: mass 0.07193524 -> 0.07848005
- link leg_l6_link: mass 0.49861272 -> 0.58491513
- link leg_r1_link: mass 1.71093008 -> 1.63861324
- link leg_r2_link: mass 0.58029165 -> 0.70575545
- link leg_r3_link: mass 4.50385993 -> 5.93791831
- link leg_r4_link: mass 1.62655699 -> 4.02498548
- link leg_r5_link: mass 0.07193524 -> 0.07848005
- link leg_r6_link: mass 0.49861272 -> 0.58491513
- link zarm_l1_link: mass 0.962 -> 0.91653322
- link zarm_l2_link: mass 0.57 -> 0.3876739
- link zarm_l3_link: mass 1.65 -> 1.77926875
- link zarm_l4_link: mass 0.429 -> 0.58507821
- link zarm_l5_link: mass 0.61 -> 0.68679955
- link zarm_l6_link: mass 0.331 -> 0.39387181
- link zarm_l7_link: mass 0.64 -> 0.61537779
- link zarm_r1_link: mass 0.962 -> 0.92062797
- link zarm_r2_link: mass 0.57 -> 0.38768053
- link zarm_r3_link: mass 1.65 -> 1.77969208
- link zarm_r4_link: mass 0.429 -> 0.58514611
- link zarm_r5_link: mass 0.61 -> 0.68473867
- link zarm_r6_link: mass 0.331 -> 0.39247462
- link zarm_r7_link: mass 0.64 -> 0.61562202
Joints:
- removed joint waist_yaw
- added joint dummy_to_base_link: type fixed, parent dummy_link, child base_link, origin xyz=0 0 0 rpy=0 0 0
- added joint head_camera: type fixed, parent zhead_2_link, child head_camera, origin xyz=0.119717018973535 0.0237514612535074 0.0262044145991832 rpy=0 0.480224871300295 0
- added joint waist_yaw_joint: type revolute, parent base_link, child waist_yaw_link, origin xyz=0 0 0.1114 rpy=0 0 0, axis 0 0 1, limit lower=-3.14159 upper=3.14159 effort=180.0 velocity=23.55
- added joint zhead_1_joint: type revolute, parent waist_yaw_link, child zhead_1_link, origin xyz=-0.003 0.0 0.3715 rpy=0 0 0, axis 0 0 1, limit lower=-1.5707963267949 upper=1.5707963267949 effort=1.5 velocity=5.23
- added joint zhead_2_joint: type revolute, parent zhead_1_link, child zhead_2_link, origin xyz=0 0 0.137954074182872 rpy=0 0 0, axis 0 1 0, limit lower=-0.349065850398866 upper=0.785398163397448 effort=12.0 velocity=5.23
- joint leg_l1_joint: origin xyz=-0.0024999 0.087 -0.066 rpy=0 0 0 -> xyz=0.0 0.095075 -0.066 rpy=0 0 0; parent torso -> base_link
- joint leg_l3_joint: origin xyz=0.000500354536093913 -0.00100000000000011 -0.1287 rpy=0 0 0 -> xyz=0 0 -0.1437 rpy=0 0 0
- joint leg_l4_joint: origin xyz=-6.87185435835039E-05 0 -0.284 rpy=0 0 0 -> xyz=0 0 -0.284 rpy=0 0 0
- joint leg_l5_joint: origin xyz=-0.000431635992531742 0 -0.346000000000001 rpy=0 0 0 -> xyz=0.002 0.0003 -0.416 rpy=0 0 0
- joint leg_r1_joint: origin xyz=-0.0024999 -0.087 -0.066 rpy=0 0 0 -> xyz=0.0 -0.095075 -0.066 rpy=0 0 0; parent torso -> base_link
- joint leg_r3_joint: origin xyz=-4.88006581312577E-05 0 -0.1287 rpy=0 0 0 -> xyz=0 0 -0.1437 rpy=0 0 0
- joint leg_r4_joint: origin xyz=0.000147138572785148 0 -0.283999982974744 rpy=0 0 0 -> xyz=0 0 -0.284 rpy=0 0 0
- joint leg_r5_joint: origin xyz=0.000119806050928577 0 -0.345999979257963 rpy=0 0 0 -> xyz=0.00199999999983541 -0.000300000028212572 -0.415999999987417 rpy=0 0 0
- joint zarm_l1_joint: origin xyz=0.003 0.28569999999999995 0.2055 rpy=0 0 0 -> xyz=-0.003 0.1737 0.2831 rpy=0 0 0; parent waist_yaw -> waist_yaw_link
- joint zarm_l2_joint: limit lower=-0.349065850398866 upper=2.0943951023932 effort=50.0 velocity=19.154 -> lower=-0.349065850398866 upper=2.0943951023932 effort=50.0 velocity=8.37333333333333; origin xyz=0 0 0 rpy=0 0 0 -> xyz=0 0.081 0 rpy=0 0 0
- joint zarm_l3_joint: limit lower=-1.5707963267949 upper=1.5707963267949 effort=39.0 velocity=18.84 -> lower=-1.5707963267949 upper=1.5707963267949 effort=36.0 velocity=9.94333333333333; origin xyz=0 0 0 rpy=0 0 0 -> xyz=0 0 -0.104 rpy=0 0 0
- joint zarm_l4_joint: limit lower=-2.61799387799149 upper=0.0 effort=50.0 velocity=18.84 -> lower=-2.61799387799149 upper=0.0 effort=50.0 velocity=8.37333333333333; origin xyz=0.0200000000000006 0 -0.283699999999996 rpy=0 0 0 -> xyz=0.02 0 -0.1797 rpy=0 0 0
- joint zarm_l5_joint: limit lower=-1.5707963267949 upper=1.5707963267949 effort=12.0 velocity=21.666 -> lower=-1.5707963267949 upper=1.5707963267949 effort=12.0 velocity=7.32666666666667; origin xyz=-0.0200000000000025 0 -0.127037274261591 rpy=0 0 0 -> xyz=-0.02 0 -0.1195 rpy=0 0 0
- joint zarm_l6_joint: limit lower=-1.30899693899575 upper=0.698131700797732 effort=12.0 velocity=21.666 -> lower=-1.30899693899575 upper=0.698131700797732 effort=12.0 velocity=7.32666666666667; origin xyz=0.000199999999999079 0 -0.106462725738415 rpy=0 0 0 -> xyz=0 0 -0.114 rpy=0 0 0
- joint zarm_l7_joint: limit lower=-0.698131700797732 upper=0.698131700797732 effort=12.0 velocity=21.666 -> lower=-0.698131700797732 upper=0.698131700797732 effort=12.0 velocity=7.32666666666667; origin xyz=0 0 -0.0210004653879916 rpy=0 0 0 -> xyz=-0.0002 0 -0.021 rpy=0 0 0
- joint zarm_r1_joint: origin xyz=0.003 -0.28569999999999995 0.2055 rpy=0 0 0 -> xyz=-0.003 -0.1737 0.2831 rpy=0 0 0; parent waist_yaw -> waist_yaw_link
- joint zarm_r2_joint: limit lower=-2.0943951023932 upper=0.349065850398866 effort=50.0 velocity=19.154 -> lower=-2.0943951023932 upper=0.349065850398866 effort=50.0 velocity=8.37333333333333; origin xyz=0 0 0 rpy=0 0 0 -> xyz=0 -0.081 0 rpy=0 0 0
- joint zarm_r3_joint: limit lower=-1.5707963267949 upper=1.5707963267949 effort=39.0 velocity=18.84 -> lower=-1.5707963267949 upper=1.5707963267949 effort=36.0 velocity=9.94333333333333; origin xyz=0 0 0 rpy=0 0 0 -> xyz=0 0 -0.104 rpy=0 0 0
- joint zarm_r4_joint: limit lower=-2.61799387799149 upper=0.0 effort=50.0 velocity=18.84 -> lower=-2.61799387799149 upper=0.0 effort=50.0 velocity=8.37333333333333; origin xyz=0.0200000000000024 0 -0.2837 rpy=0 0 0 -> xyz=0.02 0 -0.1797 rpy=0 0 0
- joint zarm_r5_joint: limit lower=-1.5707963267949 upper=1.5707963267949 effort=12.0 velocity=21.666 -> lower=-1.5707963267949 upper=1.5707963267949 effort=12.0 velocity=7.32666666666667; origin xyz=-0.0200000000000001 0 -0.127037274261587 rpy=0 0 0 -> xyz=-0.02 0 -0.1195 rpy=0 0 0
- joint zarm_r6_joint: limit lower=-0.698131700797732 upper=1.30899693899575 effort=12.0 velocity=21.666 -> lower=-0.698131700797732 upper=1.30899693899575 effort=12.0 velocity=7.32666666666667; origin xyz=0 0 -0.106462725738415 rpy=0 0 0 -> xyz=0 0 -0.114 rpy=0 0 0
- joint zarm_r7_joint: limit lower=-0.698131700797732 upper=0.698131700797732 effort=12.0 velocity=21.666 -> lower=-0.698131700797732 upper=0.698131700797732 effort=12.0 velocity=7.32666666666667; origin xyz=0 0 -0.0209999999999999 rpy=0 0 0 -> xyz=0 0 -0.022284 rpy=0 0 0
